File: doc/almost_smart_thermostat_v01.sch (EAGLE design)
At the start: 10 parts, among them IC1 L293DNE, K1 G6CU-2114P-US 3VDC

Commit message: Updated Eagle schematics and pcb design
Parts:
- added EXTERNAL, VBAT: (no value), con-lstb:MA03-1
- added FREE: (no value), con-lstb:MA07-1
- added L293_FREE: (no value), con-lstb:MA05-1
- added TERMINAL_EXTERNAL: DG300.50.-4P, heksalab:DG300.50.-4P
- K1: value G6CU-2114P-US 3VDC -> G6CU-2117P
- renumbered PHOTON_WIRES to WIRES, RESET_BUTTON to RESET
Connections:
- removed net VCC: U$1.VIN
- new net 34EN: IC1.3-4EN, L293_FREE.1
- new net 3A: IC1.3A, L293_FREE.2
- new net 3Y: IC1.3Y, L293_FREE.3
- new net 4A: IC1.4A, L293_FREE.5
- new net 4Y: IC1.4Y, L293_FREE.4
- new net A3: FREE.1, U$1.A3
- new net A4: FREE.2, U$1.A4
- new net A5: FREE.3, U$1.A5
- new net COMMON2: K13.P, TERMINAL_HEATER.P$2
- new net D7: U$1.D7, VBAT.3
- new net DAC: FREE.4, U$1.DAC
- new net E1: EXTERNAL.3, TERMINAL_EXTERNAL.P$1
- new net E2: EXTERNAL.2, TERMINAL_EXTERNAL.P$2
- new net RX: FREE.6, U$1.RX
- new net TX: FREE.7, U$1.TX
- new net VBAT: U$1.VBAT, VBAT.1
- new net WKP: FREE.5, U$1.WKP
- net CLK: now also U$1.D5; no longer U$1.D6
- net COMMON: now also K12.P; no longer K13.O, K13.P, TERMINAL_HEATER.P$2
- net CS: now also U$1.D2; no longer U$1.D3
- net DATA: now also U$1.D6; no longer U$1.D5
- net DC: now also U$1.D4; no longer U$1.D2
- net GND: now also EXTERNAL.1, TERMINAL_EXTERNAL.P$3, VBAT.2
- net NC: now also K13.O; no longer K12.S
- net NO: now also K12.S; no longer K12.P
- net RST: now also U$1.D3; no longer U$1.D4
- net VIN: now also TERMINAL_EXTERNAL.P$4, U$1.VIN
Other:
- note added: "Almost smart thermostat with additional headers made available for future upgrades/expansions. (Photon_vbat, L293_free, photon_free, external are redundant for the thermostat function)"
- moved on the sheet: IC1, RGB, SETUP
